Commit message: feat(web_ui): wheel STL mesh + interactive arm drag control in Robot Status tab
- Replace cylinder placeholders in robot.urdf with meshes/wheel.stl for all 4 wheels
- Add arm_command_topic config field (Python + YAML + TypeScript)
- Add onRobotLoaded callback to RobotModel for external robot ref access
- New InteractiveArm component: raycast to URDF joints, drag to rotate,
  publish sensor_msgs/JointState to command topic at ~20Hz
- Safety gate: drag/publish blocked until first live servo position is received,
  preventing zero-position commands on startup
- RobotStatusTab: wire InteractiveArm, show 'Waiting for servo positions…'
  until initial state arrives, then 'Drag arm joints to command position'

File: nodes/web_ui/urdf/robot.urdf (robot description, URDF)
Before this commit: robot swerve_robot, 9 links, 8 joints
Links:
- link fl_wheel_link: geometry visual mesh filename=meshes/wheel.stl
- link fr_wheel_link: geometry visual mesh filename=meshes/wheel.stl
- link rl_wheel_link: geometry visual mesh filename=meshes/wheel.stl
- link rr_wheel_link: geometry visual mesh filename=meshes/wheel.stl
