Commit message: feat(web_ui): roller wheel base model at real scale and position, wheel angles integrated live from /swerve_drive/joint_states; arm mount default matches the new body

File: nodes/web_ui/urdf/robot.urdf (robot description, URDF)
Before this commit: robot swerve_robot, 9 links, 8 joints
Links:
- link base_link: geometry visual box size=0.47 0.386 0.10
- link fl_wheel_link: geometry visual box size=0.118 0.032 0.008; visual cylinder length=0.03 radius=0.06
- link fr_wheel_link: geometry visual box size=0.118 0.032 0.008; visual cylinder length=0.03 radius=0.06
- link rl_wheel_link: geometry visual box size=0.118 0.032 0.008; visual cylinder length=0.03 radius=0.06
- link rr_wheel_link: geometry visual box size=0.118 0.032 0.008; visual cylinder length=0.03 radius=0.06
Joints:
- joint fl_drive: axis 1 0 0 -> 0 1 0
- joint fl_steer: limit lower=-3.14159 upper=3.14159 effort=10 velocity=5 -> lower=-1.5708 upper=1.5708 effort=10 velocity=5; origin xyz=0.2 0.15 -0.05 rpy=0 0 0 -> xyz=0.1525 0.1333 0.06 rpy=0 0 0
- joint fr_drive: axis 1 0 0 -> 0 1 0
- joint fr_steer: limit lower=-3.14159 upper=3.14159 effort=10 velocity=5 -> lower=-1.5708 upper=1.5708 effort=10 velocity=5; origin xyz=0.2 -0.15 -0.05 rpy=0 0 0 -> xyz=0.1525 -0.1333 0.06 rpy=0 0 0
- joint rl_drive: axis 1 0 0 -> 0 1 0
- joint rl_steer: limit lower=-3.14159 upper=3.14159 effort=10 velocity=5 -> lower=-1.5708 upper=1.5708 effort=10 velocity=5; origin xyz=-0.2 0.15 -0.05 rpy=0 0 0 -> xyz=-0.1525 0.1333 0.06 rpy=0 0 0
- joint rr_drive: axis 1 0 0 -> 0 1 0
- joint rr_steer: limit lower=-3.14159 upper=3.14159 effort=10 velocity=5 -> lower=-1.5708 upper=1.5708 effort=10 velocity=5; origin xyz=-0.2 -0.15 -0.05 rpy=0 0 0 -> xyz=-0.1525 -0.1333 0.06 rpy=0 0 0

Commit message: feat(web_ui): drop the solid placeholder body, the base shows only its 0.47 x 0.386 m footprint outline on the floor

File: nodes/web_ui/urdf/robot.urdf (robot description, URDF)
Before this commit: robot swerve_robot, 9 links, 8 joints
Links:
- link base_link: geometry visual box size=0.01 0.386 0.005; visual box size=0.01 0.386 0.005
