Commit message: feat(head): tilt range -30..+30 deg, tilt servo inverted

File: nodes/web_ui/urdf/head.urdf (robot description, URDF)
Before this commit: robot head, 9 links, 8 joints
Joints:
- joint head_tilt: limit lower=-0.5236 upper=0.7854 effort=2.0 velocity=1.0 -> lower=-0.5236 upper=0.5236 effort=2.0 velocity=1.0

Commit message: feat(head): widen head tilt range to -30..+45 deg for the reprinted mount
The task default was -30..+60 deg (D42, H6), but the Hardware section of
docs/runbooks/head-arm-calibration.md records a smaller tilt-down limit of
45 deg for the reprinted mount, so that value is used instead.

- head.urdf head_tilt limit -0.5236..0.7854 rad
- base_servos head tilt steps 1536..2389 (inverted servo: +45 deg -> 1536,
  -30 deg -> 2389); startup and mcp home tilt stay 0.5236 rad (step 1707)
- web_ui head tab tilt range [-30, 45] in client.yml, default.yaml, the
  config.py default and the HeadTab.tsx default
- tests pinned to the new range: servo steps, URDF limits, mcp_server
  kinematics (reachable floor point near 43 deg, refusal past 45 deg),
  web_ui tab defaults, the head chain override's kept limit line, and the
  frontend tilt slider default

File: nodes/web_ui/urdf/head.urdf (robot description, URDF)
Before this commit: robot head, 9 links, 8 joints
Joints:
- joint head_tilt: limit lower=-0.5236 upper=0.5236 effort=2.0 velocity=1.0 -> lower=-0.5236 upper=0.7854 effort=2.0 velocity=1.0

Commit message: feat(urdf): D435 frames on the pan/tilt head

File: nodes/web_ui/urdf/head.urdf (robot description, URDF)
Before this commit: robot head, 9 links, 8 joints
Links:
- added link d435_color_frame
- added link d435_color_optical_frame
- added link d435_depth_frame
- added link d435_depth_optical_frame
- added link d435_link; visual box size=0.090 0.025 0.025
Joints:
- added joint d435_color_joint: type fixed, parent d435_link, child d435_color_frame, origin xyz=0 -0.015 0 rpy=0 0 0
- added joint d435_color_optical_joint: type fixed, parent d435_color_frame, child d435_color_optical_frame, origin xyz=0 0 0 rpy=-1.5707963 0 -1.5707963
- added joint d435_depth_joint: type fixed, parent d435_link, child d435_depth_frame, origin xyz=0 0 0 rpy=0 0 0
- added joint d435_depth_optical_joint: type fixed, parent d435_depth_frame, child d435_depth_optical_frame, origin xyz=0 0 0 rpy=-1.5707963 0 -1.5707963
- added joint d435_joint: type fixed, parent head_link, child d435_link, origin xyz=0.02 0 0 rpy=0 0 0

Commit message: feat(realsense): D435 live bring-up, pinned topics and factory colour extrinsic
- nodes/bridges/realsense_d435/config/topics.yaml: the 26 live /head/d435/* topics with type,
  header frame_id and producing node (topic_scraper_api, 2026-10-28).
- head.urdf d435_color_joint: the factory Color-to-Depth extrinsic of the head D435 (device
  935422070045, ASIC 935723024187) in body axes; the colour imager is +15 mm in y, not -15 mm.
- docs/runbooks/d435-switchover.md Bring-up: firmware 5.16.0.1 -> 5.17.3.10 (backup, flash,
  recovery), 8086:0b07 at 5000 Mb/s, 30 min soak with zero errors, camera_info at 14.9 Hz.
- tests/test_d435_topics.py, tests/test_d435_runbook.py; the URDF FK pins in
  test_head_kinematics, test_head_urdf, test_head_arm_calib_chain and test_head_arm_fit
  follow the factory extrinsic.

File: nodes/web_ui/urdf/head.urdf (robot description, URDF)
Before this commit: robot head, 14 links, 13 joints
Joints:
- joint d435_color_joint: origin xyz=0 -0.015 0 rpy=0 0 0 -> xyz=0.0001761 0.0150171 -0.0000698 rpy=0.0082621 -0.0014919 0.0056971

Commit message: refactor(urdf): S81 remove the ToF and head camera frames

File: nodes/web_ui/urdf/head.urdf (robot description, URDF)
Before this commit: robot head, 14 links, 13 joints
Links:
- removed link head_camera_link
- removed link head_camera_optical_frame
- removed link tof_link
- removed link tof_optical_frame
Joints:
- removed joint head_camera_joint
- removed joint head_camera_optical_joint
- removed joint tof_joint
- removed joint tof_optical_joint
